Commit message: Reformat code, add depth transport, fix container build

File: urdf/include/depthai_macro.urdf.xacro (robot description, xacro)
@@ -1,10 +1,23 @@
 <?xml version="1.0"?>
 <robot name="depthai_camera" xmlns:xacro="http://ros.org/wiki/xacro">
-<xacro:macro name="depthai_camera" params="camera_name camera_model parent base_frame cam_pos_x cam_pos_y cam_pos_z cam_roll cam_pitch cam_yaw">
+<xacro:macro name="depthai_camera" params="camera_name camera_model parent base_frame
+                                           cam_pos_x cam_pos_y cam_pos_z
+                                           cam_roll cam_pitch cam_yaw
+                                           r:=0.8 g:=0.8 b:=0.8 a:=0.8">
     <xacro:property name="M_PI"     value="3.1415926535897931" />
     <xacro:property name="model"    value="${camera_model}" />
+    <xacro:property name="has_imu" value="false" />
     <!-- <xacro:if value="${model == 'BW1098OAK'}">
     </xacro:if> -->
     <xacro:property name="baseline" value="0.075" />
+    <xacro:if value="${model == 'OAK-D'}">
+      <xacro:property name="has_imu" value="true" />
+      <xacro:property name="imu_offset_x" value="0.0" />
+      <xacro:property name="imu_offset_y" value="-0.015" />
+      <xacro:property name="imu_offset_z" value="-0.013662" />
+      <xacro:property name="imu_r" value="0" />
+      <xacro:property name="imu_p" value="1.5708" />
+      <xacro:property name="imu_y" value="0" />
+    </xacro:if>
     <!-- base_link of the sensor-->
     <link name="${base_frame}"/>
@@ -22,5 +35,5 @@
             </geometry>
             <material name="mat">
-                <color rgba="0.8 0.8 0.8 0.8"/>
+                <color rgba="${r} ${g} ${b} ${a}"/>
             </material>
         </visual>
@@ -32,13 +45,15 @@
     </joint>
 <!-- IMU -->
-    <link name="${ camera_name}_imu_frame" />
-    <joint name="${ camera_name}_imu_joint" type="fixed">
-        <parent link="${base_frame}"/>
-        <child link="${camera_name}_imu_frame"/>
-        <origin xyz="0 0 0" rpy="-${M_PI/2} 0 -${M_PI/2}" />
-    </joint>
+    <xacro:if value="${has_imu}">
+        <link name="${camera_name}_imu_frame" />
+        <joint name="${camera_name}_imu_joint" type="fixed">
+            <parent link="${base_frame}"/>
+            <child link="${camera_name}_imu_frame"/>
+            <origin xyz="${imu_offset_x} ${imu_offset_y} ${imu_offset_z}" rpy="${imu_r} ${imu_p} ${imu_y}" />
+        </joint>
+    </xacro:if>
 <!-- RGB Camera -->
-    <link name="${ camera_name}_rgb_camera_frame" />
-    <joint name="${ camera_name}_rgb_camera_joint" type="fixed">
+    <link name="${camera_name}_rgb_camera_frame" />
+    <joint name="${camera_name}_rgb_camera_joint" type="fixed">
         <parent link="${base_frame}"/>
         <child link="${camera_name}_rgb_camera_frame"/>
